Commit message: chore: meshes + urdf

File: stretch_description/urdf/xacro/stretch_base_imu.xacro (robot description, xacro)
@@ -10,5 +10,5 @@
       <origin xyz="0 0 0" rpy="0 0 0" />
       <geometry>
-        <mesh filename="package://stretch_description/meshes/base_imu.STL" />
+        <mesh filename="file://$(find stretch_description)/meshes/base_imu.STL" />
       </geometry>
       <material name="">
@@ -19,5 +19,5 @@
       <origin xyz="0 0 0" rpy="0 0 0" />
       <geometry>
-        <mesh filename="package://stretch_description/meshes/base_imu.STL" />
+        <mesh filename="file://$(find stretch_description)/meshes/base_imu.STL" />
       </geometry>
     </collision>
