Commit message: chore: gazebo base control

File: stretch_description/urdf/xacro/stretch_description_RE2V0_tool_stretch_gripper.xacro (robot description, xacro)
@@ -1,10 +1,11 @@
 <?xml version="1.0"?>
 <robot xmlns:xacro="http://www.ros.org/wiki/xacro" name="stretch">
-  <xacro:include filename="stretch_main.xacro" />
-  <xacro:include filename="stretch_aruco.xacro" />
+  <xacro:include filename="$(find stretch_description)/urdf/xacro/stretch_main.xacro" />
+  <!-- <xacro:include filename="stretch_aruco.xacro" />
   <xacro:include filename="stretch_d435i.xacro" />
   <xacro:include filename="stretch_laser_range_finder.xacro" />
   <xacro:include filename="stretch_base_imu.xacro" />
   <xacro:include filename="stretch_respeaker.xacro" />
-  <xacro:include filename="stretch_gripper_with_puller.xacro" />
+  <xacro:include filename="stretch_gripper_with_puller.xacro" /> -->
+  <xacro:include filename="$(find stretch_description)/urdf/xacro/stretch.gazebo" />
 </robot>

File: stretch_description/urdf/xacro/stretch_main.xacro (robot description, xacro)
@@ -3,5 +3,5 @@
   <xacro:property name="M_PI" value="3.1415926535897931" />
   <xacro:property name="joint_damping" value="21.75"/>
-  <xacro:property name="joint_friction" value="10.48"/>
+  <xacro:property name="joint_friction" value="0.1"/>
   <xacro:property name="joint_spring_stiffness" value="0"/>
   <xacro:property name="joint_spring_reference" value="0"/>
@@ -22,5 +22,5 @@
     </visual>
     <collision>
-      <origin xyz="0 0 0" rpy="0 0 0" />
+      <origin xyz="0 0 0.1" rpy="0 0 0" />
       <geometry>
         <mesh filename="file://$(find stretch_description)/meshes/base_link_collision.STL" />
@@ -30,10 +30,10 @@
   <link name="link_right_wheel">
     <inertial>
-      <origin xyz="0 0 0.02765" rpy="0 0 0" />
+      <origin xyz="0 0 0.02765" rpy="0.0 3.1416 0" />
       <mass value="0.20773" />
       <inertia ixx="5.4E-05" ixy="0" ixz="0" iyy="5.4E-05" iyz="0" izz="5.1E-05" />
     </inertial>
     <visual>
-      <origin xyz="0 0 0" rpy="0 0 0" />
+      <origin xyz="0 0 0" rpy="0.0 3.1416 0" />
       <geometry>
         <mesh filename="file://$(find stretch_description)/meshes/link_right_wheel.STL" />
@@ -44,12 +44,20 @@
     </visual>
     <collision>
-      <origin xyz="0 0 0" rpy="0 0 0" />
-      <geometry>
-        <mesh filename="file://$(find stretch_description)/meshes/link_right_wheel_collision.STL" />
-      </geometry>
-    </collision>
-  </link>
-  <joint name="joint_right_wheel" type="continuous">
-    <origin xyz="0 -0.17035 0.0508" rpy="-1.5708 1.2717E-16 4.8006E-17" />
+      <origin xyz="0 0 -0.0125" rpy="0.0 0.0 0" />
+      <geometry>
+        <cylinder radius="0.05" length="0.025"/>
+      </geometry>
+      <!-- <surface>
+        <friction>
+          <ode>
+            <mu>100.01</mu>
+            <mu2>100.01</mu2>
+          </ode>
+        </friction>
+      </surface> -->
+    </collision>
+  </link>
+  <joint name="joint_right_wheel" type="fixed">
+    <origin xyz="0 -0.17035 0.0508" rpy="1.5708 1.5708 4.8006E-17" />
     <parent link="base_link" />
     <child link="link_right_wheel" />
@@ -64,5 +72,5 @@
     </inertial>
     <visual>
-      <origin xyz="0 0 0" rpy="0 0 0" />
+      <origin xyz="0 0 0" rpy="0.0 3.1416 0" />
       <geometry>
         <mesh filename="file://$(find stretch_description)/meshes/link_left_wheel.STL" />
@@ -73,12 +81,20 @@
     </visual>
     <collision>
-      <origin xyz="0 0 0" rpy="0 0 0" />
-      <geometry>
-        <mesh filename="file://$(find stretch_description)/meshes/link_left_wheel_collision.STL" />
-      </geometry>
-    </collision>
-  </link>
-  <joint name="joint_left_wheel" type="continuous">
-    <origin xyz="0 0.17035 0.0508" rpy="-1.5708 2.6317E-16 -8.2057E-19" />
+      <origin xyz="0 0 0.0125" rpy="0 0 0" />
+      <geometry>
+        <cylinder radius="0.05" length="0.025"/>
+      </geometry>
+      <!-- <surface>
+        <friction>
+          <ode>
+            <mu>100.0</mu>
+            <mu2>100.0</mu2>
+          </ode>
+        </friction>
+      </surface> -->
+    </collision>
+  </link>
+  <joint name="joint_left_wheel" type="fixed">
+    <origin xyz="0 0.17035 0.0508" rpy="${M_PI/2} ${M_PI/2} -8.2057E-19" />
     <parent link="base_link" />
     <child link="link_left_wheel" />
@@ -179,9 +195,7 @@
     <child link="link_lift" />
     <axis xyz="0 0 1" />
-    <!-- for now: hand copied range_m: from lift: from ~/repos/stretch_fleet/stretch-re1-1001/stretch_re1_factory_params.yaml -->
-    <!--<limit effort="100" lower="0.0" upper="1.095" velocity="1.0"/>-->
-    <!-- copied value did not reach the top of mesh model with GUI sliders and RViz -->
     <limit effort="100" lower="0.0" upper="1.1" velocity="1.0"/>
   </joint>
+  <!--
   <link name="link_arm_l4">
     <inertial>
@@ -239,5 +253,4 @@
     <child link="link_arm_l3" />
     <axis xyz="0 0 1" />
-    <!-- 0.13 = 0.52/4-->
     <limit effort="100" lower="0.0" upper="0.13" velocity="1.0"/>
   </joint>
@@ -269,5 +282,4 @@
     <child link="link_arm_l2" />
     <axis xyz="0 0 1" />
-    <!-- 0.13 = 0.52/4-->
     <limit effort="100" lower="0.0" upper="0.13" velocity="1.0"/>
   </joint>
@@ -299,5 +311,4 @@
     <child link="link_arm_l1" />
     <axis xyz="0 0 1" />
-    <!-- 0.13 = 0.52/4-->
     <limit effort="100" lower="0.0" upper="0.13" velocity="1.0"/>
   </joint>
@@ -329,5 +340,4 @@
     <child link="link_arm_l0" />
     <axis xyz="0 0 1" />
-    <!-- 0.13 = 0.52/4-->
     <limit effort="100" lower="0.0" upper="0.13" velocity="1.0"/>
   </joint>
@@ -359,10 +369,4 @@
     <child link="link_wrist_yaw" />
     <axis xyz="0 0 -1" />
-    <!--
-      stowed to front ~225 deg: 3.15159 x 1.25 = 3.9395
-      using 4.0
-      stowed to back ~100 deg:  100 / 180 x 3.14159 = 1.7453
-      using -1.75
-    -->
     <limit effort="100" lower="-1.75" upper="4.0" velocity="1.0"/>
   </joint>
@@ -422,5 +426,4 @@
     <child link="link_head_pan" />
     <axis xyz="0 0 1" />
-    <!-- unconstrained range for now -->
     <limit effort="100" lower="-3.9" upper="1.5" velocity="1.0"/>
   </joint>
@@ -452,6 +455,5 @@
     <child link="link_head_tilt" />
     <axis xyz="0 0 1" />
-    <!-- unconstrained range for now -->
     <limit effort="100" lower="-1.53" upper="0.79" velocity="1.0"/>
-  </joint>
+  </joint> -->
 </robot>
