Commit message: chor: simple stretch urdf plannar move

File: stretch_description/urdf/xacro/stretch_d435i.xacro (robot description, xacro)
@@ -3,5 +3,5 @@
   <xacro:arg name="use_nominal_extrinsics" default="true"/>
   <xacro:arg name="add_plug" default="false"/>
-  <xacro:include filename="d435i/_d435i.urdf.xacro"/>
+  <xacro:include filename="$(find realsense2_description)/urdf/_d435i.urdf.xacro"/>
   <!-- xyz = "
        depth (- recessed into head / + protruding from front)

File: stretch_description/urdf/xacro/stretch_dex_wrist.xacro (robot description, xacro)
@@ -20,5 +20,5 @@
       <origin xyz="0 0 0" rpy="0 0 0" />
       <geometry>
-        <mesh filename="file://$(find stretch_description)/meshes/link_wrist_yaw_bottom_collision.STL" />
+        <mesh filename="file://$(find stretch_description)/meshes/link_wrist_yaw_bottom.STL" />
       </geometry>
     </collision>
@@ -48,9 +48,9 @@
       <origin xyz="0 0 0" rpy="0 0 0" />
       <geometry>
-        <mesh filename="file://$(find stretch_description)/meshes/link_wrist_pitch_collision.STL" />
-      </geometry>
-    </collision>
-  </link>
-  <joint name="joint_wrist_pitch" type="revolute">
+        <mesh filename="file://$(find stretch_description)/meshes/link_wrist_pitch.STL" />
+      </geometry>
+    </collision>
+  </link>
+  <joint name="joint_wrist_pitch" type="fixed">
     <origin xyz="0 -0.0195500000000002 -0.0247499999999984" rpy="1.5707963267949 -8.12895570882604E-15 -3.14159265358979" />
     <parent link="link_wrist_yaw_bottom" />
@@ -77,9 +77,9 @@
       <origin xyz="0 0 0" rpy="0 0 0" />
       <geometry>
-        <mesh filename="file://$(find stretch_description)/meshes/link_wrist_roll_collision.STL" />
-      </geometry>
-    </collision>
-  </link>
-  <joint name="joint_wrist_roll" type="revolute">
+        <mesh filename="file://$(find stretch_description)/meshes/link_wrist_roll.STL" />
+      </geometry>
+    </collision>
+  </link>
+  <joint name="joint_wrist_roll" type="fixed">
     <origin xyz="-0.0188587444076125 -0.0239999999998942 0.01955" rpy="3.14159265358979 1.5707963267949 0" />
     <parent link="link_wrist_pitch" />
@@ -106,5 +106,5 @@
       <origin xyz="0 0 0" rpy="0 0 0" />
       <geometry>
-        <mesh filename="file://$(find stretch_description)/meshes/link_straight_gripper_collision.STL" />
+        <mesh filename="file://$(find stretch_description)/meshes/link_straight_gripper.STL" />
       </geometry>
     </collision>
@@ -134,9 +134,9 @@
       <origin xyz="0 0 0" rpy="0 0 0" />
       <geometry>
-        <mesh filename="file://$(find stretch_description)/meshes/link_gripper_finger_right_collision.STL" />
-      </geometry>
-    </collision>
-  </link>
-  <joint name="joint_gripper_finger_right" type="revolute">
+        <mesh filename="file://$(find stretch_description)/meshes/link_gripper_finger_right.STL" />
+      </geometry>
+    </collision>
+  </link>
+  <joint name="joint_gripper_finger_right" type="fixed">
     <origin xyz="-0.018599 0.003 0.033689" rpy="1.5708 1.5708 0" />
     <parent link="link_straight_gripper" />
@@ -163,5 +163,5 @@
       <origin xyz="0 0 0" rpy="0 0 0" />
       <geometry>
-        <mesh filename="file://$(find stretch_description)/meshes/link_gripper_fingertip_right_collision.STL" />
+        <mesh filename="file://$(find stretch_description)/meshes/link_gripper_fingertip_right.STL" />
       </geometry>
     </collision>
@@ -191,9 +191,9 @@
       <origin xyz="0 0 0" rpy="1.5707963267948966 0 0" />
       <geometry>
-        <mesh filename="file://$(find stretch_description)/meshes/link_gripper_finger_left_collision.STL" />
-      </geometry>
-    </collision>
-  </link>
-  <joint name="joint_gripper_finger_left" type="revolute">
+        <mesh filename="file://$(find stretch_description)/meshes/link_gripper_finger_left.STL" />
+      </geometry>
+    </collision>
+  </link>
+  <joint name="joint_gripper_finger_left" type="fixed">
     <origin xyz="0.018599 0.003 0.033689" rpy="1.5708 -1.5708 0" />
     <parent link="link_straight_gripper" />
@@ -220,5 +220,5 @@
       <origin xyz="0 0 0" rpy="0 0 0" />
       <geometry>
-        <mesh filename="file://$(find stretch_description)/meshes/link_gripper_fingertip_left_collision.STL" />
+        <mesh filename="file://$(find stretch_description)/meshes/link_gripper_fingertip_left.STL" />
       </geometry>
     </collision>

File: stretch_description/urdf/xacro/stretch_gripper.xacro (robot description, xacro)
@@ -20,5 +20,5 @@
       <origin xyz="0 0 0" rpy="0 0 0" />
       <geometry>
-        <mesh filename="file://$(find stretch_description)/meshes/link_gripper_collision.STL" />
+        <mesh filename="file://$(find stretch_description)/meshes/link_gripper.STL" />
       </geometry>
     </collision>
@@ -50,9 +50,9 @@
       <origin xyz="0 0 0" rpy="0 0 0" />
       <geometry>
-        <mesh filename="file://$(find stretch_description)/meshes/link_gripper_finger_left_collision.STL" scale="${scale_finger_length} 1.0 1.0"/>
+        <mesh filename="file://$(find stretch_description)/meshes/link_gripper_finger_left.STL" scale="${scale_finger_length} 1.0 1.0"/>
       </geometry>
     </collision>
   </link>
-  <joint name="joint_gripper_finger_left" type="revolute">
+  <joint name="joint_gripper_finger_left" type="fixed">
     <origin xyz="-0.047231 -0.010151 -0.04679" rpy="2.1762E-15 0.5236 3.1416" />
     <parent link="link_gripper" />
@@ -79,5 +79,5 @@
       <origin xyz="0 0 0" rpy="0 0 0" />
       <geometry>
-        <mesh filename="file://$(find stretch_description)/meshes/link_gripper_fingertip_left_collision.STL" />
+        <mesh filename="file://$(find stretch_description)/meshes/link_gripper_fingertip_left.STL" />
       </geometry>
     </collision>
@@ -107,9 +107,9 @@
       <origin xyz="0 0 0" rpy="0 0 0" />
       <geometry>
-        <mesh filename="file://$(find stretch_description)/meshes/link_gripper_finger_right_collision.STL" scale="${scale_finger_length} 1.0 1.0"/>
+        <mesh filename="file://$(find stretch_description)/meshes/link_gripper_finger_right.STL" scale="${scale_finger_length} 1.0 1.0"/>
       </geometry>
     </collision>
   </link>
-  <joint name="joint_gripper_finger_right" type="revolute">
+  <joint name="joint_gripper_finger_right" type="fixed">
     <origin xyz="-0.047231 0.010049 -0.04679" rpy="3.1416 -0.5236 1.2943E-15" />
     <parent link="link_gripper" />
@@ -136,5 +136,5 @@
       <origin xyz="0 0 0" rpy="0 0 0" />
       <geometry>
-        <mesh filename="file://$(find stretch_description)/meshes/link_gripper_fingertip_right_collision.STL" />
+        <mesh filename="file://$(find stretch_description)/meshes/link_gripper_fingertip_right.STL" />
       </geometry>
     </collision>

File: stretch_description/urdf/xacro/stretch_gripper_with_puller.xacro (robot description, xacro)
@@ -20,5 +20,5 @@
       <origin xyz="0 0 0" rpy="0 0 0" />
       <geometry>
-        <mesh filename="file://$(find stretch_description)/meshes/link_gripper_collision.STL" />
+        <mesh filename="file://$(find stretch_description)/meshes/link_gripper.STL" />
       </geometry>
     </collision>
@@ -78,9 +78,9 @@
       <origin xyz="0 0 0" rpy="0 0 0" />
       <geometry>
-        <mesh filename="file://$(find stretch_description)/meshes/link_gripper_finger_left_collision.STL" scale="${scale_finger_length} 1.0 1.0"/>
+        <mesh filename="file://$(find stretch_description)/meshes/link_gripper_finger_left.STL" scale="${scale_finger_length} 1.0 1.0"/>
       </geometry>
     </collision>
   </link>
-  <joint name="joint_gripper_finger_left" type="revolute">
+  <joint name="joint_gripper_finger_left" type="fixed">
     <origin xyz="-0.047231 -0.010151 -0.04679" rpy="2.1762E-15 0.5236 3.1416" />
     <parent link="link_gripper" />
@@ -107,5 +107,5 @@
       <origin xyz="0 0 0" rpy="0 0 0" />
       <geometry>
-        <mesh filename="file://$(find stretch_description)/meshes/link_gripper_fingertip_left_collision.STL" />
+        <mesh filename="file://$(find stretch_description)/meshes/link_gripper_fingertip_left.STL" />
       </geometry>
     </collision>
@@ -135,9 +135,9 @@
       <origin xyz="0 0 0" rpy="0 0 0" />
       <geometry>
-        <mesh filename="file://$(find stretch_description)/meshes/link_gripper_finger_right_collision.STL" scale="${scale_finger_length} 1.0 1.0"/>
+        <mesh filename="file://$(find stretch_description)/meshes/link_gripper_finger_right.STL" scale="${scale_finger_length} 1.0 1.0"/>
       </geometry>
     </collision>
   </link>
-  <joint name="joint_gripper_finger_right" type="revolute">
+  <joint name="joint_gripper_finger_right" type="fixed">
     <origin xyz="-0.047231 0.010049 -0.04679" rpy="3.1416 -0.5236 1.2943E-15" />
     <parent link="link_gripper" />
@@ -164,5 +164,5 @@
       <origin xyz="0 0 0" rpy="0 0 0" />
       <geometry>
-        <mesh filename="file://$(find stretch_description)/meshes/link_gripper_fingertip_right_collision.STL" />
+        <mesh filename="file://$(find stretch_description)/meshes/link_gripper_fingertip_right.STL" />
       </geometry>
     </collision>

File: stretch_description/urdf/xacro/stretch_laser_range_finder.xacro (robot description, xacro)
@@ -19,5 +19,5 @@
       <origin xyz="0 0 0" rpy="0 0 0" />
       <geometry>
-        <mesh filename="file://$(find stretch_description)/meshes/laser_collision.STL" />
+        <mesh filename="file://$(find stretch_description)/meshes/laser.STL" />
       </geometry>
     </collision>

File: stretch_description/urdf/xacro/stretch_main.xacro (robot description, xacro)
@@ -3,5 +3,5 @@
   <xacro:property name="M_PI" value="3.1415926535897931" />
   <xacro:property name="joint_damping" value="21.75"/>
-  <xacro:property name="joint_friction" value="0.1"/>
+  <xacro:property name="joint_friction" value="10.48"/>
   <xacro:property name="joint_spring_stiffness" value="0"/>
   <xacro:property name="joint_spring_reference" value="0"/>
@@ -22,7 +22,7 @@
     </visual>
     <collision>
-      <origin xyz="0 0 0.1" rpy="0 0 0" />
-      <geometry>
-        <mesh filename="file://$(find stretch_description)/meshes/base_link_collision.STL" />
+      <origin xyz="0 0 0" rpy="0 0 0" />
+      <geometry>
+        <mesh filename="file://$(find stretch_description)/meshes/base_link.STL" />
       </geometry>
     </collision>
@@ -30,10 +30,10 @@
   <link name="link_right_wheel">
     <inertial>
-      <origin xyz="0 0 0.02765" rpy="0.0 3.1416 0" />
+      <origin xyz="0 0 0.02765" rpy="0 0 0" />
       <mass value="0.20773" />
       <inertia ixx="5.4E-05" ixy="0" ixz="0" iyy="5.4E-05" iyz="0" izz="5.1E-05" />
     </inertial>
     <visual>
-      <origin xyz="0 0 0" rpy="0.0 3.1416 0" />
+      <origin xyz="0 0 0" rpy="0 0 0" />
       <geometry>
         <mesh filename="file://$(find stretch_description)/meshes/link_right_wheel.STL" />
@@ -44,20 +44,12 @@
     </visual>
     <collision>
-      <origin xyz="0 0 -0.0125" rpy="0.0 0.0 0" />
-      <geometry>
-        <cylinder radius="0.05" length="0.025"/>
-      </geometry>
-      <!-- <surface>
-        <friction>
-          <ode>
-            <mu>100.01</mu>
-            <mu2>100.01</mu2>
-          </ode>
-        </friction>
-      </surface> -->
+      <origin xyz="0 0 0" rpy="0 0 0" />
+      <geometry>
+        <mesh filename="file://$(find stretch_description)/meshes/link_right_wheel.STL" />
+      </geometry>
     </collision>
   </link>
   <joint name="joint_right_wheel" type="fixed">
-    <origin xyz="0 -0.17035 0.0508" rpy="1.5708 1.5708 4.8006E-17" />
+    <origin xyz="0 -0.17035 0.0508" rpy="-1.5708 1.2717E-16 4.8006E-17" />
     <parent link="base_link" />
     <child link="link_right_wheel" />
@@ -72,5 +64,5 @@
     </inertial>
     <visual>
-      <origin xyz="0 0 0" rpy="0.0 3.1416 0" />
+      <origin xyz="0 0 0" rpy="0 0 0" />
       <geometry>
         <mesh filename="file://$(find stretch_description)/meshes/link_left_wheel.STL" />
@@ -81,20 +73,12 @@
     </visual>
     <collision>
-      <origin xyz="0 0 0.0125" rpy="0 0 0" />
-      <geometry>
-        <cylinder radius="0.05" length="0.025"/>
-      </geometry>
-      <!-- <surface>
-        <friction>
-          <ode>
-            <mu>100.0</mu>
-            <mu2>100.0</mu2>
-          </ode>
-        </friction>
-      </surface> -->
+      <origin xyz="0 0 0" rpy="0 0 0" />
+      <geometry>
+        <mesh filename="file://$(find stretch_description)/meshes/link_left_wheel.STL" />
+      </geometry>
     </collision>
   </link>
   <joint name="joint_left_wheel" type="fixed">
-    <origin xyz="0 0.17035 0.0508" rpy="${M_PI/2} ${M_PI/2} -8.2057E-19" />
+    <origin xyz="0 0.17035 0.0508" rpy="-1.5708 2.6317E-16 -8.2057E-19" />
     <parent link="base_link" />
     <child link="link_left_wheel" />
@@ -158,5 +142,5 @@
       <origin xyz="0 0 0" rpy="0 0 0" />
       <geometry>
-        <mesh filename="file://$(find stretch_description)/meshes/link_mast_collision.STL" />
+        <mesh filename="file://$(find stretch_description)/meshes/link_mast.STL" />
       </geometry>
     </collision>
@@ -186,16 +170,18 @@
       <origin xyz="0 0 0" rpy="0 0 0" />
       <geometry>
-        <mesh filename="file://$(find stretch_description)/meshes/link_lift_collision.STL" />
-      </geometry>
-    </collision>
-  </link>
-  <joint name="joint_lift" type="prismatic">
-    <origin xyz="-0.037385 0.1666 0" rpy="-1.5708 1.5708 0" />
+        <mesh filename="file://$(find stretch_description)/meshes/link_lift.STL" />
+      </geometry>
+    </collision>
+  </link>
+  <joint name="joint_lift" type="fixed">
+    <origin xyz="-0.037385 1.0 0.0" rpy="-1.5708 1.5708 0" />
     <parent link="link_mast" />
     <child link="link_lift" />
     <axis xyz="0 0 1" />
+    <!-- for now: hand copied range_m: from lift: from ~/repos/stretch_fleet/stretch-re1-1001/stretch_re1_factory_params.yaml -->
+    <!--<limit effort="100" lower="0.0" upper="1.095" velocity="1.0"/>-->
+    <!-- copied value did not reach the top of mesh model with GUI sliders and RViz -->
     <limit effort="100" lower="0.0" upper="1.1" velocity="1.0"/>
   </joint>
-  <!--
   <link name="link_arm_l4">
     <inertial>
@@ -216,5 +202,5 @@
       <origin xyz="0 0 0" rpy="0 0 0" />
       <geometry>
-        <mesh filename="file://$(find stretch_description)/meshes/link_arm_l4_collision.STL" />
+        <mesh filename="file://$(find stretch_description)/meshes/link_arm_l4.STL" />
       </geometry>
     </collision>
@@ -244,13 +230,14 @@
       <origin xyz="0 0 0" rpy="0 0 0" />
       <geometry>
-        <mesh filename="file://$(find stretch_description)/meshes/link_arm_l3_collision.STL" />
-      </geometry>
-    </collision>
-  </link>
-  <joint name="joint_arm_l3" type="prismatic">
+        <mesh filename="file://$(find stretch_description)/meshes/link_arm_l3.STL" />
+      </geometry>
+    </collision>
+  </link>
+  <joint name="joint_arm_l3" type="fixed">
     <origin xyz="0 0 0.013" rpy="7.68831233799385E-30 2.36716479416092E-30 2.29652732251143E-17" />
     <parent link="link_arm_l4" />
     <child link="link_arm_l3" />
     <axis xyz="0 0 1" />
+    <!-- 0.13 = 0.52/4-->
     <limit effort="100" lower="0.0" upper="0.13" velocity="1.0"/>
   </joint>
@@ -273,13 +260,14 @@
       <origin xyz="0 0 0" rpy="0 0 0" />
       <geometry>
-        <mesh filename="file://$(find stretch_description)/meshes/link_arm_l2_collision.STL" />
-      </geometry>
-    </collision>
-  </link>
-  <joint name="joint_arm_l2" type="prismatic">
+        <mesh filename="file://$(find stretch_description)/meshes/link_arm_l2.STL" />
+      </geometry>
+    </collision>
+  </link>
+  <joint name="joint_arm_l2" type="fixed">
     <origin xyz="0 0 0.013" rpy="0 1.57655765344625E-30 -1.66533453693773E-16" />
     <parent link="link_arm_l3" />
     <child link="link_arm_l2" />
     <axis xyz="0 0 1" />
+    <!-- 0.13 = 0.52/4-->
     <limit effort="100" lower="0.0" upper="0.13" velocity="1.0"/>
   </joint>
@@ -302,13 +290,14 @@
       <origin xyz="0 0 0" rpy="0 0 0" />
       <geometry>
-        <mesh filename="file://$(find stretch_description)/meshes/link_arm_l1_collision.STL" />
-      </geometry>
-    </collision>
-  </link>
-  <joint name="joint_arm_l1" type="prismatic">
+        <mesh filename="file://$(find stretch_description)/meshes/link_arm_l1.STL" />
+      </geometry>
+    </collision>
+  </link>
+  <joint name="joint_arm_l1" type="fixed">
     <origin xyz="0 0 0.0129999999999981" rpy="-7.63746778746202E-30 -7.88860905221012E-31 1.11022302462516E-16" />
     <parent link="link_arm_l2" />
     <child link="link_arm_l1" />
     <axis xyz="0 0 1" />
+    <!-- 0.13 = 0.52/4-->
     <limit effort="100" lower="0.0" upper="0.13" velocity="1.0"/>
   </joint>
@@ -331,13 +320,14 @@
       <origin xyz="0 0 0" rpy="0 0 0" />
       <geometry>
-        <mesh filename="file://$(find stretch_description)/meshes/link_arm_l0_collision.STL" />
-      </geometry>
-    </collision>
-  </link>
-  <joint name="joint_arm_l0" type="prismatic">
+        <mesh filename="file://$(find stretch_description)/meshes/link_arm_l0.STL" />
+      </geometry>
+    </collision>
+  </link>
+  <joint name="joint_arm_l0" type="fixed">
     <origin xyz="0 0 -0.0137499999991968" rpy="7.63746778746202E-30 -3.80121128864402E-15 2.62707547767438E-15" />
     <parent link="link_arm_l1" />
     <child link="link_arm_l0" />
     <axis xyz="0 0 1" />
+    <!-- 0.13 = 0.52/4-->
     <limit effort="100" lower="0.0" upper="0.13" velocity="1.0"/>
   </joint>
@@ -360,13 +350,19 @@
       <origin xyz="0 0 0" rpy="0 0 0" />
       <geometry>
-        <mesh filename="file://$(find stretch_description)/meshes/link_wrist_yaw_collision.STL" />
-      </geometry>
-    </collision>
-  </link>
-  <joint name="joint_wrist_yaw" type="revolute">
-    <origin xyz="0.0830000000000654 -0.0307500000000129 0" rpy="1.5708 4.2595E-14 2.6415E-15"/>
+        <mesh filename="file://$(find stretch_description)/meshes/link_wrist_yaw.STL" />
+      </geometry>
+    </collision>
+  </link>
+  <joint name="joint_wrist_yaw" type="fixed">
+    <origin xyz="0.0830000000000654 -0.0307500000000129 0" rpy="3.1416 4.2595E-14 2.6415E-15"/>
     <parent link="link_arm_l0" />
     <child link="link_wrist_yaw" />
     <axis xyz="0 0 -1" />
+    <!--
+      stowed to front ~225 deg: 3.15159 x 1.25 = 3.9395
+      using 4.0
+      stowed to back ~100 deg:  100 / 180 x 3.14159 = 1.7453
+      using -1.75
+    -->
     <limit effort="100" lower="-1.75" upper="4.0" velocity="1.0"/>
   </joint>
@@ -389,5 +385,5 @@
       <origin xyz="0 0 0" rpy="0 0 0" />
       <geometry>
-        <mesh filename="file://$(find stretch_description)/meshes/link_head_collision.STL" />
+        <mesh filename="file://$(find stretch_description)/meshes/link_head.STL" />
       </geometry>
     </collision>
@@ -417,13 +413,14 @@
       <origin xyz="0 0 0" rpy="0 0 0" />
       <geometry>
-        <mesh filename="file://$(find stretch_description)/meshes/link_head_pan_collision.STL" />
-      </geometry>
-    </collision>
-  </link>
-  <joint name="joint_head_pan" type="revolute">
+        <mesh filename="file://$(find stretch_description)/meshes/link_head_pan.STL" />
+      </geometry>
+    </collision>
+  </link>
+  <joint name="joint_head_pan" type="fixed">
     <origin xyz="0.135 0.0731000000000001 -0.00319621125547975" rpy="0 0 1.5707963267949" />
     <parent link="link_head" />
     <child link="link_head_pan" />
     <axis xyz="0 0 1" />
+    <!-- unconstrained range for now -->
     <limit effort="100" lower="-3.9" upper="1.5" velocity="1.0"/>
   </joint>
@@ -446,14 +443,80 @@
       <origin xyz="0 0 0" rpy="0 0 0" />
       <geometry>
-        <mesh filename="file://$(find stretch_description)/meshes/link_head_tilt_collision.STL" />
-      </geometry>
-    </collision>
-  </link>
-  <joint name="joint_head_tilt" type="revolute">
+        <mesh filename="file://$(find stretch_description)/meshes/link_head_tilt.STL" />
+      </geometry>
+    </collision>
+  </link>
+  <joint name="joint_head_tilt" type="fixed">
     <origin xyz="-0.00130000001785262 0.0277624999926072 -0.0533107920897029" rpy="1.5707963267949 3.36459255518345E-15 -8.42914893687103E-17" />
     <parent link="link_head_pan" />
     <child link="link_head_tilt" />
     <axis xyz="0 0 1" />
+    <!-- unconstrained range for now -->
     <limit effort="100" lower="-1.53" upper="0.79" velocity="1.0"/>
-  </joint> -->
+  </joint>
+  <link name="link_tray">
+    <visual>
+      <origin xyz="0 0 0" rpy="0 0 0" />
+      <geometry>
+        <mesh filename="file://$(find stretch_description)/meshes/tray.dae" />
+      </geometry>
+    </visual>
+    <collision>
+      <origin xyz="0 0 0" rpy="0 0 0" />
+      <geometry>
+        <mesh filename="file://$(find stretch_description)/meshes/tray.dae" />
+      </geometry>
+    </collision>
+  </link>
+  <joint name="joint_tray_base" type="fixed">
+    <origin xyz="0.0 0.0 0.5" rpy="0.0 0.0 1.57" />
+    <parent link="base_link" />
+    <child link="link_tray" />
+    <axis xyz="0 0 1" />
+  </joint>
+  <!-- pills -->
+  <link name="link_pills">
+    <visual>
+      <origin xyz="0 0 0" rpy="0 0 0" />
+      <geometry>
+        <mesh filename="file://$(find stretch_description)/meshes/pills.dae" />
+      </geometry>
+    </visual>
+  </link>
+  <joint name="joint_pills_tray" type="fixed">
+    <origin xyz="0.02 0.05 0.01" rpy="0.0 0.0 0.0" />
+    <parent link="link_tray" />
+    <child link="link_pills" />
+    <axis xyz="0 0 1" />
+  </joint>
+  <!-- pill dispenser -->
+  <link name="link_pills_dispenser">
+    <visual>
+      <origin xyz="0 0 0" rpy="1.57 0 0" />
+      <geometry>
+        <mesh filename="file://$(find stretch_description)/meshes/pills_dispenser.dae" scale="0.3 0.3 0.3" />
+      </geometry>
+    </visual>
+  </link>
+  <joint name="joint_pills_dispenser_tray" type="fixed">
+    <origin xyz="0.01 -0.02 -0.04" rpy="0.0 0.0 0.0" />
+    <parent link="link_tray" />
+    <child link="link_pills_dispenser" />
+    <axis xyz="0 0 1" />
+  </joint>
+  <!-- water bottle -->
+  <link name="link_water_bottle">
+    <visual>
+      <origin xyz="0 0 0" rpy="1.57 0 0" />
+      <geometry>
+        <mesh filename="file://$(find stretch_description)/meshes/water_bottle.dae" scale="0.5 0.5 0.5"/>
+      </geometry>
+    </visual>
+  </link>
+  <joint name="joint_water_bottle_tray" type="fixed">
+    <origin xyz="-0.125 -0.03 0.01" rpy="0.0 0.0 0.0" />
+    <parent link="link_tray" />
+    <child link="link_water_bottle" />
+    <axis xyz="0 0 1" />
+  </joint>
 </robot>
