Commit message: chore: base footprint in urdf

File: stretch_gz_sim/urdf/stretch_re1/stretch_main.xacro (robot description, xacro)
@@ -2,4 +2,16 @@
 <robot xmlns:xacro="http://www.ros.org/wiki/xacro" name="stretch_main">
   <xacro:property name="M_PI" value="3.1415926535897931" />
+  <link name="base_footprint" />
+  <joint
+    name="joint_base_footprint"
+    type="fixed">
+    <origin
+      xyz="0 0 0"
+      rpy="0 0 0" />
+    <parent
+      link="base_footprint" />
+    <child
+      link="base_link" />
+  </joint>
   <link
     name="base_link">

Commit message: [Update]: Stretch RE1 version 2.0

File: stretch_gz_sim/urdf/stretch_re1/stretch_main.xacro (robot description, xacro)
@@ -2,16 +2,4 @@
 <robot xmlns:xacro="http://www.ros.org/wiki/xacro" name="stretch_main">
   <xacro:property name="M_PI" value="3.1415926535897931" />
-  <link name="base_footprint" />
-  <joint
-    name="joint_base_footprint"
-    type="fixed">
-    <origin
-      xyz="0 0 0"
-      rpy="0 0 0" />
-    <parent
-      link="base_footprint" />
-    <child
-      link="base_link" />
-  </joint>
   <link
     name="base_link">
